File: 5_electronics.kicad_pcb (KiCad board)
At the start: 2 copper layers, 0 parts

Commit message: Update routing
Parts:
- added BT1: Battery_Cell, Battery:BatteryHolder_Keystone_103_1x20mm, F.Cu at (70.8, 52.2)
- added CAMERA1: Conn_01x15, Connector_PinHeader_2.54mm:PinHeader_1x15_P2.54mm_Vertical, F.Cu at (116.0, 57.6)
- added E_Paper1: Conn_01x08, Connector_PinHeader_2.54mm:PinHeader_1x08_P2.54mm_Vertical, F.Cu at (100.0, 78.4)
- added FAN1: Conn_01x02, Connector_PinHeader_2.54mm:PinHeader_1x02_P2.54mm_Vertical, F.Cu at (57.0, 42.0)
- added I2C_SENSOR_CONNECTOR1: Conn_01x04, Connector_PinHeader_2.54mm:PinHeader_1x04_P2.54mm_Vertical, F.Cu at (57.0, 81.0)
- added INA219_Sensor1: Conn_01x06, Connector_PinHeader_2.54mm:PinHeader_1x06_P2.54mm_Vertical, F.Cu at (67.0, 63.8)
- added J1: Conn_02x20_Odd_Even, Connector_PinHeader_2.54mm:PinHeader_2x20_P2.54mm_Vertical, F.Cu at (47.5, 39.9)
- added PIR_Sensor1: Conn_01x04, Connector_PinHeader_2.54mm:PinHeader_1x04_P2.54mm_Vertical, F.Cu at (56.5, 57.0)
- added Temperature&Humidity_Sensor1: Conn_01x04, Connector_PinHeader_2.54mm:PinHeader_1x04_P2.54mm_Vertical, F.Cu at (82.0, 80.5)
Routing:
- net GND: track 0.00 -> 156.1 mm
- net +3V3: track 0.00 -> 90.4 mm
- net I2C_SDA: track 0.00 -> 44.1 mm
- net I2C_SCL: track 0.00 -> 44.1 mm
- net +3.3V: track 0.00 -> 31.6 mm
- net BAT+: track 0.00 -> 23.7 mm
- net +5V: track 0.00 -> 9.73 mm
- added copper zone on B.Cu, net GND
Other:
- board outline added: 81 x 65.5 mm
